Commit message: done

File: description/robot.urdf.xacro (robot description, xacro)
@@ -3,3 +3,7 @@
     <!-- Example link -->
     <xacro:include filename="robot_core.xacro"/>
+    <xacro:include filename="robot_control.xacro"/>
+    <xacro:include filename="lidar.xacro"/>
+    <!--  <xacro:include filename="camera.xacro"/> -->
+    <xacro:include filename="depth_camera.xacro"/>
 </robot>

File: description/robot_core.xacro (robot description, xacro)
@@ -50,4 +50,7 @@
         </xacro:inertial_box>
     </link>
+    <gazebo reference="chassis">
+        <material>Gazebo/SkyBlue</material>
+    </gazebo>
     <!-- left wheel link -->
     <joint name="left_wheel_joint" type="continuous">
@@ -73,4 +76,7 @@
         </xacro:inertial_cylinder>
     </link>
+    <gazebo reference="left_wheel_link">
+        <material>Gazebo/Green</material>
+    </gazebo>
     <!-- right wheel link -->
     <joint name="right_wheel_joint" type="continuous">
@@ -96,5 +102,8 @@
         </xacro:inertial_cylinder>
     </link>
-    <!-- right wheel link -->
+    <gazebo reference="right_wheel_link">
+        <material>Gazebo/Green</material>
+    </gazebo>
+    <!-- caster wheel link -->
     <joint name="caster_wheel_joint" type="fixed">
         <parent link="chassis"/>
@@ -118,3 +127,8 @@
         </xacro:inertial_sphere>
     </link>
+    <gazebo reference="caster_wheel_link">
+        <material>Gazebo/Green</material>
+        <mu1 value="0.001"/>
+        <mu2 value="0.001"/>
+    </gazebo>
 </robot>
